File: hardware/shutdown_circuit.kicad_sch (KiCad schematic)
At the start: 43 parts, among them J1 Screw_Terminal_01x06, J2 Raspberry_Pi_4, J3 6W Header, J4 6W Header, Q1 Q_NMOS_GDS, Q2 Q_Dual_PNP, Q3 Q_PMOS_SDG, U1 SFH617A-1, U2 LM2576HVS-3.3, U3 DS1307+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

Commit message: Updated for HAT MKII & new firmware
Parts:
- removed D10, D2, D4, D5, D7: 1N4007, pilot_footprints:1N4007FLTR, symbol Diode:1N4007
- removed D3: 1N5822, pilot_footprints:1N4007FLTR, symbol Diode:1N5822
- removed D8, D9: RB520S30T1G, pilot_footprints:schottky_diodes, symbol Device:D_Schottky
- removed Q2: Q_Dual_PNP, pilot_footprints:pnp_pair, symbol Device:Q_Dual_NPN_PNP_E1B1C2E2B2C1
- removed Q3: Q_PMOS_SDG, pilot_footprints:zvd_mosfet, symbol Device:Q_PMOS_SDG
- removed R12: 47k, Resistor_SMD:R_0603_1608Metric_Pad0.98x0.95mm_HandSolder, symbol Device:R_US
- removed R6: 1k, Resistor_SMD:R_0603_1608Metric_Pad0.98x0.95mm_HandSolder, symbol Device:R_US
- removed R8: 4k7, Resistor_SMD:R_0603_1608Metric_Pad0.98x0.95mm_HandSolder, symbol Device:R_US
- removed R9: 10k, Resistor_SMD:R_0603_1608Metric_Pad0.98x0.95mm_HandSolder, symbol Device:R_US
- removed U4: SFH617A-1, Package_DIP:DIP-4_W7.62mm, symbol Isolator:SFH617A-1
- added C?: 100nF, symbol Device:C_Small
- added C?: 10uF, symbol Device:C_Small
- added C?: 100uF, pilot_footprints:100uF_Cap, symbol Device:C_Polarized
- added D? (x3): Schottky, symbol Device:D_Schottky_Small
- added D? (x3): RB520S30T1G, symbol Device:D_Schottky_Small
- added D?: G_LED, LED_SMD:LED_0603_1608Metric_Pad1.05x0.95mm_HandSolder, symbol Device:LED
- added F?: Fuse, symbol Device:Fuse_Small
- added Q2: IRF9540N, symbol Device:Q_PMOS_GDS
- added R?: 100, Resistor_SMD:R_0603_1608Metric_Pad0.98x0.95mm_HandSolder, symbol Device:R_US
- added R?: 4k7, Resistor_SMD:R_0603_1608Metric_Pad0.98x0.95mm_HandSolder, symbol Device:R_US
- added R?: 1k, Resistor_SMD:R_0603_1608Metric_Pad0.98x0.95mm_HandSolder, symbol Device:R_US
- added U?: SFH617A-1, Package_DIP:DIP-4_W7.62mm, symbol Isolator:SFH617A-1
- D6: value LED -> R_LED
- J1: value Screw_Terminal_01x06 -> Screw Terminal
- Q1: value Q_NMOS_GDS -> DMN63D8
- R1: value 15k -> 10k
- R3: value 4k7 -> 10k
Connections:
- net +12v_ACC: now also R1.2, R?.1
- net +12v_BAT: now also F?.1; no longer D1.2 (A), R1.2
- net +3v3: now also D?.2 (A), D?.2 (A), R?.1
- net ACC_Opto: now also D?.1 (K), D?.1 (K), R?.2, U?.4
- net ATTINY_VCC: now also C?.1, C?.1, D?.1 (K)
- net GND: now also C1.2, J1.6 (Pin_6), R2.1, U2.3 (GND), U2.5 (~{ON}/OFF), C?.2, C?.2, C?.2, D?.1 (K), D?.2 (A), U?.2, U?.3; no longer R3.1
- net MISO: no longer U5.6 (PB1)
- net RESET: now also D?.2 (A)
- net at D1.1 (K): now also Q2.3 (S); no longer U2.1 (VIN)
- net at L1.1, U2.2 (OUT): now also D?.1 (K)
- net at R3.2: no longer R2.1
- net at J2.16 (GPIO23): now also D?.2 (A)
- net at U5.3 (XTAL2/PB4): now also D?.2 (A)
- net STAT_LED: now reaches U5.2 (XTAL1/PB3)
- net STAT_LED: now also R?.1
- net MOSFET_CTRL renamed FET_CTRL
- net FET_CTRL: now also D?.1 (K)
- new net: D1.2 (A), F?.2
- new net: C?.1, Q2.2 (D), U2.1 (VIN)
- new net: D?.2 (A), R?.2
- new net: R?.2, U?.1
- new net: Q1.2 (D), Q2.1 (G), R3.1
- no-connect marks 24 -> 23
Other:
- note added: ""The Brains""
- note added: "Power Supply"
- note added: "Shutoff Detection"
- note removed: "RPi 5v ZVD"
- note removed: "Shutdown Controller"
- moved on the sheet: BT1, C1, D1, D6, J1, J3, L1, Q1, R1, R2, R7, U2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

Commit message: Updated schematic & schematic screenshots
Connections:
- net RESET: no longer D?.2 (A)
- net STAT_LED: now also U5.6 (PB1); no longer U5.2 (XTAL1/PB3)
- new net: D?.2 (A), U5.2 (XTAL1/PB3)
Other:
- moved on the sheet: D?
Changed lines of the file:
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@@
   (junction (at 236.22 142.24) (diameter 0) (color 0 0 0 0)
-  )
-  (junction (at 130.3528 85.852) (diameter 0) (color 0 0 0 0)
   )
   (junction (at 78.8416 62.5856) (diameter 0) (color 0 0 0 0)
@@
     (stroke (width 0) (type default) (color 0 0 0 0))
   )
-  (wire (pts (xy 116.2812 85.852) (xy 125.2728 85.852))
+  (wire (pts (xy 116.2812 80.772) (xy 125.2728 80.772))
     (stroke (width 0) (type default) (color 0 0 0 0))
   )
@@
     (stroke (width 0) (type default) (color 0 0 0 0))
   )
-  (wire (pts (xy 130.3528 85.852) (xy 130.3528 93.472))
-    (stroke (width 0) (type default) (color 0 0 0 0))
-  )
   (polyline (pts (xy 15.24 143.51) (xy 15.24 153.67))
     (stroke (width 0) (type default) (color 0 0 0 0))
@@
     (stroke (width 0) (type default) (color 0 0 0 0))
   )
-  (wire (pts (xy 115.9256 80.772) (xy 130.3528 80.772))
+  (wire (pts (xy 115.9256 68.072) (xy 130.3528 68.072))
     (stroke (width 0) (type default) (color 0 0 0 0))
   )
@@
     (stroke (width 0) (type default) (color 0 0 0 0))
   )
-  (wire (pts (xy 115.9764 93.472) (xy 130.3528 93.472))
+  (wire (pts (xy 115.9764 85.852) (xy 130.3528 85.852))
     (stroke (width 0) (type default) (color 0 0 0 0))
   )
@@
     (effects (font (size 1.27 1.27)) (justify right bottom))
   )
-  (label "RESET" (at 115.9764 93.472 0)
+  (label "RESET" (at 115.9764 85.852 0)
     (effects (font (size 1.27 1.27)) (justify left bottom))
   )
@@
     (effects (font (size 1.27 1.27)) (justify right bottom))
   )
-  (label "ACC_Opto" (at 116.2812 85.852 0)
+  (label "ACC_Opto" (at 116.2812 80.772 0)
     (effects (font (size 1.27 1.27)) (justify left bottom))
   )
@@
     (effects (font (size 1.27 1.27)) (justify right bottom))
   )
-  (label "STAT_LED" (at 115.9256 80.772 0)
+  (label "STAT_LED" (at 115.9256 68.072 0)
     (effects (font (size 1.27 1.27)) (justify left bottom))
   )
@@
     (pin "1")
   )
-  (symbol (lib_id "Device:D_Schottky_Small") (at 127.8128 85.852 0) (unit 1)
+  (symbol (lib_id "Device:D_Schottky_Small") (at 127.8128 80.772 0) (unit 1)
     (in_bom yes) (on_board yes)
-    (property "Reference" "D?" (id 0) (at 126.1618 87.122 0)
+    (property "Reference" "D?" (id 0) (at 131.572 81.8896 0)
       (effects (font (size 1.27 1.27)) (justify right))
     )
-    (property "Value" "Schottky" (id 1) (at 129.3368 89.027 0)
+    (property "Value" "Schottky" (id 1) (at 130.302 83.3628 0)
       (effects (font (size 1.27 1.27)) (justify right))
     )
-    (property "Footprint" "" (id 2) (at 127.8128 85.852 90)
-      (effects (font (size 1.27 1.27)) hide)
-    )
-    (property "Datasheet" "~" (id 3) (at 127.8128 85.852 90)
-      (effects (font (size 1.27 1.27)) hide)
-    )
+    (property "Footprint" "" (id 2) (at 127.8128 80.772 90)
+      (effects (font (size 1.27 1.27)) hide)
+    )
+    (property "Datasheet" "~" (id 3) (at 127.8128 80.772 90)
+      (effects (font (size 1.27 1.27)) hide)
+    )

Commit message: PILOT Drive HAT MKII
Parts:
- removed BT1: Battery_Cell, Battery:BatteryHolder_Keystone_106_1x20mm, symbol Device:Battery_Cell
- removed J1: Screw Terminal, pilot_footprints:screw_term_6, symbol Connector:Screw_Terminal_01x06
- added BT1: BLP2032SM-GTR, pilot_footprints:RTC_Battery_Holder, symbol RTC_Battery_Holder:BLP2032SM-GTR
- added D2: ESD12VD3B, Diode_SMD:D_SOD-323, symbol Diode:1N4007
- added D3: SMLJ60S10, Diode_SMD:D_SMC_Handsoldering, symbol Diode:1N4007
- added D4: CDSOD323-T15S, Diode_SMD:D_SOD-323F, symbol Diode:1N4007
- added F2: 3414.0124.26, Fuse:Fuse_0402_1005Metric_Pad0.77x0.64mm_HandSolder, symbol Device:Fuse_Small
- added J1: 284391-7, pilot_footprints:Screw_Term, symbol Connector:Screw_Terminal_01x07
- C1: footprint pilot_footprints:100uF_Cap -> pilot_footprints:1000uF_10v
- C2: renamed from C?; footprint pilot_footprints:100uF_Cap -> pilot_footprints:100uF_35v
- C3, C4: renamed from C?; footprint (none) -> Capacitor_SMD:C_0402_1005Metric_Pad0.74x0.62mm_HandSolder
- D1: value 1N4007 -> SMLJ60S10; footprint pilot_footprints:1N4007FLTR -> Diode_SMD:D_SMC_Handsoldering
- D10, D11, D12: renamed from D?; footprint (none) -> pilot_footprints:3v3_TVS
- D5: renamed from D?; value Schottky -> B340LB-13-F; footprint (none) -> Diode_SMD:D_SMC_Handsoldering
- D7, D8: renamed from D?; value Schottky -> RB520S30T1G; footprint (none) -> pilot_footprints:3v3_TVS
- F1: renamed from F?; value Fuse -> 3414.0124.26; footprint (none) -> Fuse:Fuse_0402_1005Metric_Pad0.77x0.64mm_HandSolder
- L1: footprint pilot_footprints:induct_100uH -> pilot_footprints:100uH_Inductor
- Q1: value DMN63D8 -> DMN63D8L-7; footprint Package_TO_SOT_THT:TO-220-3_Vertical -> pilot_footprints:N_FET
- Q2: footprint (none) -> pilot_footprints:P_FET
- R1, R10, R11, R13, R14, R15, R16, R2, R3, R4, R5, R7: footprint Resistor_SMD:R_0603_1608Metric_Pad0.98x0.95mm_HandSolder -> Resistor_SMD:R_0402_1005Metric_Pad0.72x0.64mm_HandSolder
- R6, R8, R9: renamed from R?; footprint Resistor_SMD:R_0603_1608Metric_Pad0.98x0.95mm_HandSolder -> Resistor_SMD:R_0402_1005Metric_Pad0.72x0.64mm_HandSolder
- U1: value SFH617A-1 -> SFH617A-1X007T; footprint Package_DIP:DIP-4_W7.62mm -> pilot_footprints:Optocoupler
- U3: value DS1307+ -> DS1307Z+; footprint Package_DIP:DIP-8_W7.62mm -> pilot_footprints:DS1307Z+T&R
- U4: renamed from U?; value SFH617A-1 -> SFH617A-1X007T; footprint Package_DIP:DIP-4_W7.62mm -> pilot_footprints:Optocoupler
- U5: value ATtiny85-20P -> ATtiny85-20SUR; footprint Package_SO:SOIC-8W_5.3x5.3mm_P1.27mm -> pilot_footprints:ATTINY_SUR
- U6: footprint Package_SO:TSSOP-8_4.4x3mm_P0.65mm -> pilot_footprints:CAT24C128YI
- Y1: footprint Crystal:Crystal_SMD_3215-2Pin_3.2x1.5mm -> pilot_footprints:RTC_Crystal
- gave numbers to parts that had none: 1
Connections:
- net +5v_ZVD is gone; now on net +5v: J2.2 (5V), J2.4 (5V), U3.8 (VCC)
- net STAT_LED is gone; now on net MISO: R9.1, U5.6 (PB1)
- net +12v_ACC: now also F2.2, J1.1 (Pin_1); no longer R1.2
- net +12v_BAT: now also J1.2 (Pin_2)
- net +12v_HL: now also J1.4 (Pin_4)
- net +5v: now also J1.5 (Pin_5)
- net BACKUP_BTN: now also J1.6 (Pin_6)
- net GND: now also BT1.-, D2.2 (A), D4.2 (A), J1.7 (Pin_7)
- net RTC_Bat: now also BT1.+
- net at J4.6 (Pin_6), R15.2, U6.8 (VCC): now also D12.1 (K)
- net at D1.1 (K): now also Q2.2 (S), R3.2, D4.1 (K); no longer Q2.3 (S)
- net +12v_OUT: now reaches C2.1, U2.1 (VIN)
- net +12v_OUT: now also Q2.3 (D), J1.3 (Pin_3); no longer Q2.2 (D)
- new net: D2.1 (K), D3.1 (K), R1.2
- new net: D3.2 (A), F2.1
Other:
- moved on the sheet: C1, C2, D1, D12, D5, D6, F1, L1, Q1, Q2, R1, R2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
